File: pcb/v0.2/toasterBoard.kicad_pcb (KiCad board)
At the start: 2 copper layers, 66 x 44.4 mm, 37 parts, among them IC1 ATMEGA328P_TQFP, IC2 MIC5205, IC3 MAX6675, IC4 BLE112-A, J1 MICROUSB, J2 TOASTER, J3 CC_ISP, K1 S116S02F, M3 VAL**, P1 AVR_ISP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

Commit message: small changes
Parts:
- IC1: value ATMEGA328P_TQFP -> ATMEGA328P
Changed lines of the file:
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@@
       (effects (font (size 1.524 1.524) (thickness 0.3048)))
     )
-    (fp_text value ATMEGA328P_TQFP (at -1.99898 -6.49986 315) (layer F.SilkS) hide
+    (fp_text value ATMEGA328P (at -6.986639 1.670328 405) (layer F.SilkS)
       (effects (font (size 1.524 1.524) (thickness 0.3048)))
     )
@@
   (module ED110 (layer F.Cu)
     (at 225.806 133.604 270)
-    (fp_text reference J2 (at 6.35 6.604 270) (layer F.SilkS)
-      (effects (font (size 1.524 1.524) (thickness 0.3048)))
-    )
-    (fp_text value TOASTER (at -2.54 -5.588 270) (layer F.SilkS)
-      (effects (font (size 1.524 1.524) (thickness 0.3048)))
-    )
+    (fp_text reference J2 (at 6.35 6.604 270) (layer F.SilkS) hide
+      (effects (font (size 1.524 1.524) (thickness 0.3048)))
+    )
+    (fp_text value TOASTER (at 9.271 -0.2794 360) (layer F.SilkS)
+      (effects (font (size 1.524 1.524) (thickness 0.3048)))
+    )
