File: pcb/v0.2/toasterBoard.kicad_pcb (KiCad board)
At the start: 2 copper layers, 66 x 44.4 mm, 37 parts, among them IC1 ATMEGA328P, IC2 MIC5205, IC3 MAX6675, IC4 BLE112-A, J1 MICROUSB, J2 TOASTER, J3 CC_ISP, K1 S116S02F, M3 VAL**, P1 AVR_ISP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

Commit message: small changes to board
Parts:
- moved S1 11.0 mm to (267.1, 131.4), turned to 180 degrees
- moved R9 5.68 mm to (260.1, 123.7), turned to 270 degrees
- moved LED2 4.92 mm to (258.6, 123.7), turned to 90 degrees
- moved C4 2.82 mm to (260.1, 120.4)
- moved F1 2.31 mm to (263.0, 119.1)
- moved IC2 1.60 mm to (255.8, 119.8), turned to 270 degrees
Routing:
- net GND: track 187.1 -> 179.9 mm, vias 3 -> 1
- net /RESET: track 45.3 -> 46.9 mm
- net VCC: track 124.9 -> 125.6 mm
